File: hardware/stamp_s3a_interposer/stamp_s3a_interposer_pcba.kicad_pcb (KiCad board)
At the start: 2 copper layers, 110 x 72 mm, 38 parts

Commit message: Finalize compact Stamp-S3A interposer manufacturing files
Parts:
- C1: value 470uF/10V LOGIC -> 470uF/16V LOGIC
- C3: value 1000uF/10V SERVO -> 1000uF/35V SERVO
- J_AMP_SIG: value AMP:LRC,BCLK,DIN,GAIN -> AMP:LRC,BCLK,DIN,GND
- J_PWR_LOGIC: value INPUT:5V_LOGIC,GND -> INPUT:COMMON_5V,GND
- J_PWR_SERVO: value INPUT:5V_SERVO,GND -> INPUT:COMMON_5V,GND
- J_SERVO_5V_OUT: value SERVO:5V,GND -> SERVO:COMMON_5V,GND
Connections:
- C3 pad 1: +5V_SERVO -> +5V_LOGIC
- J_PWR_SERVO pad 1: +5V_SERVO -> +5V_LOGIC
- J_SERVO_5V_OUT pad 1: +5V_SERVO -> +5V_LOGIC
Routing:
- net +5V_LOGIC: track 147.9 -> 181.4 mm
- net +5V_SERVO: track 23.7 -> 0.00 mm
Changed lines of the file:
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@@
 			)
 		)
-		(property "Value" "470uF/10V LOGIC"
+		(property "Value" "470uF/16V LOGIC"
 			(at 2.5 6.25 0)
 			(layer "F.Fab")
@@
 			)
 		)
-		(property "Value" "INPUT:5V_SERVO,GND"
+		(property "Value" "INPUT:COMMON_5V,GND"
 			(at 1.25 4.6 0)
 			(layer "F.Fab")
@@
 			(remove_unused_layers no)
 			(roundrect_rratio 0.147059)
-			(net "+5V_SERVO")
+			(net "+5V_LOGIC")
 		)
 		(pad "2" thru_hole oval
@@
 			)
 		)
-		(property "Value" "1000uF/10V SERVO"
+		(property "Value" "1000uF/35V SERVO"
 			(at 2.5 7.5 0)
 			(layer "F.Fab")
@@
 			(remove_unused_layers no)
 			(roundrect_rratio 0.104167)
-			(net "+5V_SERVO")
+			(net "+5V_LOGIC")
 		)
 		(pad "2" thru_hole circle
@@
 			)
 		)
-		(property "Value" "AMP:LRC,BCLK,DIN,GAIN"
+		(property "Value" "AMP:LRC,BCLK,DIN,GND"
 			(at 3.75 4.6 90)
 			(layer "F.Fab")
@@
 			)
 		)
-		(property "Value" "INPUT:5V_LOGIC,GND"
+		(property "Value" "INPUT:COMMON_5V,GND"
 			(at 1.25 4.6 0)
 			(layer "F.Fab")
@@
 			)
 		)
-		(property "Value" "SERVO:5V,GND"
+		(property "Value" "SERVO:COMMON_5V,GND"
 			(at 1.25 4.6 0)
 			(layer "F.Fab")
@@
 			(remove_unused_layers no)
 			(roundrect_rratio 0.147059)
-			(net "+5V_SERVO")
+			(net "+5V_LOGIC")
 		)
 		(pad "2" thru_hole oval
@@
 	)
 	(segment
+		(start 94 75)
+		(end 95.7378 76.7378)
+		(width 1)
+		(layer "F.Cu")
+		(net "+5V_LOGIC")
+	)
+	(segment
 		(start 86.2517 62)
 		(end 85.2517 63)
@@
 	)
 	(segment
+		(start 95.7378 76.7378)
+		(end 103.2622 76.7378)
+		(width 1)
+		(layer "F.Cu")
+		(net "+5V_LOGIC")
+	)
+	(segment
 		(start 98 49)
 		(end 99.2244 47.7756)
@@
 	)
 	(segment
+		(start 103.2622 76.7378)
+		(end 105 75)
+		(width 1)
+		(layer "F.Cu")
+		(net "+5V_LOGIC")
+	)
+	(segment
 		(start 26.5 15)
 		(end 27.9273 13.5727)
@@
 	)
 	(segment
+		(start 105 68)
+		(end 105 75)
+		(width 1)
+		(layer "B.Cu")
+		(net "+5V_LOGIC")
+	)
+	(segment
+		(start 108 65)
+		(end 105 68)
+		(width 1)
+		(layer "B.Cu")
+		(net "+5V_LOGIC")
+	)
+	(segment
+		(start 94 75)
+		(end 90 71.7483)
+		(width 1)
+		(layer "B.Cu")
+		(net "+5V_LOGIC")
+	)
+	(segment
 		(start 85.2517 71.7483)
 		(end 85.2517 64.9557)
@@
 	)
 	(segment
+		(start 90 71.7483)
+		(end 85.2517 71.7483)
+		(width 1)
+		(layer "B.Cu")
+		(net "+5V_LOGIC")
+	)
+	(segment
 		(start 68.35 42.7421)
 		(end 68.35 65.125)
@@
 	)
 	(segment
-		(start 94 75)
-		(end 95.7378 76.7378)
-		(width 1)
-		(layer "F.Cu")
-		(net "+5V_SERVO")
-	)
-	(segment
-		(start 95.7378 76.7378)
-		(end 103.2622 76.7378)
-		(width 1)
-		(layer "F.Cu")
-		(net "+5V_SERVO")
-	)
-	(segment
-		(start 103.2622 76.7378)
-		(end 105 75)
-		(width 1)
-		(layer "F.Cu")
-		(net "+5V_SERVO")
-	)
-	(segment
-		(start 105 68)
-		(end 105 75)
-		(width 1)
-		(layer "B.Cu")
-		(net "+5V_SERVO")
-	)
-	(segment
-		(start 108 65)
-		(end 105 68)
-		(width 1)
-		(layer "B.Cu")
-		(net "+5V_SERVO")
-	)
-	(segment
