File: hardware/stamp_s3a_interposer/stamp_s3a_interposer_pcba.kicad_sch (KiCad schematic)
At the start: 38 parts

Commit message: Finalize compact Stamp-S3A interposer manufacturing files
Parts:
- C1: value 470uF/10V LOGIC -> 470uF/16V LOGIC
- C3: value 1000uF/10V SERVO -> 1000uF/35V SERVO
- J_AMP_SIG: value AMP:LRC,BCLK,DIN,GAIN -> AMP:LRC,BCLK,DIN,GND
- J_PWR_LOGIC: value INPUT:5V_LOGIC,GND -> INPUT:COMMON_5V,GND
- J_PWR_SERVO: value INPUT:5V_SERVO,GND -> INPUT:COMMON_5V,GND
- J_SERVO_5V_OUT: value SERVO:5V,GND -> SERVO:COMMON_5V,GND
Connections:
- net +5V_SERVO is gone; now on net +5V_LOGIC: C3.1, J_PWR_SERVO.1 (Pin_1), J_SERVO_5V_OUT.1 (Pin_1)
Other:
- note added: "C1 470uF/16V LOGIC"
- note added: "C3 1000uF/35V SERVO"
- note added: "Servo V+ and logic/audio use the common +5V_LOGIC rail; both power-input XH connectors are parallel."
- note removed: "C1 470uF/10V LOGIC"
- note removed: "C3 1000uF/10V SERVO"
- note removed: "Servos connect to the PCA9685 module 3-pin outputs; servo V+ is the separate +5V_SERVO rail."
Changed lines of the file:
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@@
 		(comment 1 "Genuine JST XH; pin order is the harness contract")
 		(comment 2 "Stamp-S3A sockets are mirrored on the carrier PCB")
-		(comment 3 "Logic 5 V and servo 5 V are separate rails")
+		(comment 3 "Logic/audio and servo loads share one external 5 V rail")
 		(comment 4 "Functional schematic matched to production PCB netlist")
 	)
@@
 			)
 		)
-		(property "Value" "INPUT:5V_LOGIC,GND"
+		(property "Value" "INPUT:COMMON_5V,GND"
 			(at 27.94 30.48 0.0000)
 			(effects
@@
 			)
 		)
-		(property "Value" "470uF/10V LOGIC"
+		(property "Value" "470uF/16V LOGIC"
 			(at 53.34 34.29 0.0000)
 			(effects
@@
 			)
 		)
-		(property "Value" "INPUT:5V_SERVO,GND"
+		(property "Value" "INPUT:COMMON_5V,GND"
 			(at 27.94 77.47 0.0000)
 			(effects
@@
 			)
 		)
-		(property "Value" "1000uF/10V SERVO"
+		(property "Value" "1000uF/35V SERVO"
 			(at 53.34 82.55 0.0000)
 			(effects
@@
 			)
 		)
-		(property "Value" "SERVO:5V,GND"
+		(property "Value" "SERVO:COMMON_5V,GND"
 			(at 87.63 77.47 0.0000)
 			(effects
@@
 			)
 		)
-		(property "Value" "AMP:LRC,BCLK,DIN,GAIN"
+		(property "Value" "AMP:LRC,BCLK,DIN,GND"
 			(at 149.86 127 0.0000)
 			(effects
@@
 		)
 	)
-	(global_label "+5V_SERVO"
+	(global_label "+5V_LOGIC"
 		(shape bidirectional)
 		(at 15.24 82.55 0)
@@
 		)
 	)
-	(global_label "+5V_SERVO"
+	(global_label "+5V_LOGIC"
 		(shape bidirectional)
 		(at 53.34 71.12 0)
@@
 		)
 	)
-	(global_label "+5V_SERVO"
+	(global_label "+5V_LOGIC"
 		(shape bidirectional)
 		(at 74.93 82.55 0)
@@
 		)
 	)
-	(text "Servos connect to the PCA9685 module 3-pin outputs; servo V+ is the separate +5V_SERVO rail."
+	(text "Servo V+ and logic/audio use the common +5V_LOGIC rail; both power-input XH connectors are parallel."
 		(exclude_from_sim no)
 		(at 105 241 0.0000)
@@
 		)
 	)
-	(text "C1  470uF/10V LOGIC"
+	(text "C1  470uF/16V LOGIC"
 		(exclude_from_sim no)
 		(at 59 28 0.0000)
@@
 		)
 	)
-	(text "C3  1000uF/10V SERVO"
+	(text "C3  1000uF/35V SERVO"
 		(exclude_from_sim no)
 		(at 59 76 0.0000)
